File: camera module.sch (KiCad schematic (older format))
At the start: 165 parts, among them J1 Conn_01x02, J10 Conn_01x04, J11 Conn_01x05, J12 Conn_01x06, J13 Conn_01x02, J14 USB_A, J16 Conn_01x02, J17 USB_B_Micro, J18 Conn_01x03, J19 Conn_01x02, J2 USB_OTG, J20 Conn_01x02, J21 Conn_01x02, J22 Conn_01x02, J23 Conn_01x02, J24 Conn_01x05, J3 Conn_01x15, J4 Conn_02x15_Counter_Clockwise, J5 HDMI_A, J6 Conn_01x15, J7 Conn_01x02, J8 HDMI_A, J9 HDMI_A, Q1 DMMT5401-7-F, Q10 DMG2305UX, Q11 DMMT5401-7-F, Q12 DMG2305UX, Q7 DMMT5401-7-F, Q8 DMG2305UX, Q9 DMMT5401-7-F, SW1 SW_SPST, U1 TPS563208, U10 HDMIULC6-4SC6, U11 AP2331SA-7, U12 FSUSB42UMX, U3 LTC3406ES5-1.2, U4 PAM2306AYPKE, U5 TLV70228_SOT23-5, U6 EM6K34T2CR, U7 LSM6DS3, U8 SIT8008AI-73-XXS-33.333333E, U9 XC6222B181MR-G

Commit message: Add files via upload
Parts:
- removed D4, D5: LED, LEDs:LED_0805_HandSoldering, symbol Device:LED
- removed J11: Conn_01x05, Pin_Headers:Pin_Header_Straight_1x05_Pitch2.54mm, symbol Connector_Generic:Conn_01x05
- removed J?: Conn_01x06, symbol Connector_Generic:Conn_01x06
- removed R23, R26: 470R, Resistors_SMD:R_0603_HandSoldering, symbol Device:R
- added J?: Conn_01x08, symbol Connector_Generic:Conn_01x08
- added J?: Conn_01x04, Pin_Headers:Pin_Header_Straight_1x04_Pitch2.54mm, symbol Connector_Generic:Conn_01x04
Connections:
- net labels added: CAM0_IO1, CAM0_offboard_IO1, CAM0_onboard_IO1, CAM1_IO1
- net labels removed: CAM0_CK, CAM0_offboard_CK, CAM1_CK, CAM1_CLK, GPIO28, GPIO29
- wire segments 598 -> 582
Changed lines of the file:
@@
 Text GLabel 19750 2600 2    50   Input ~ 0
 GPIO27
-Text GLabel 21200 1550 1    50   Input ~ 0
+Text GLabel 21450 1650 0    50   Input ~ 0
 CD1_SDA
-Text GLabel 21100 1550 1    50   Input ~ 0
+Text GLabel 21450 1750 0    50   Input ~ 0
 CD1_SCL
 Text GLabel 21450 1850 0    50   Input ~ 0
-CAM1_CLK
+CAM1_IO1
 Text GLabel 21450 1950 0    50   Input ~ 0
 CAM1_IO0
 Text GLabel 21450 2050 0    50   Input ~ 0
-CAM0_CK
+CAM0_IO1
 Text GLabel 21450 2150 0    50   Input ~ 0
 CAM0_IO0
@@
 $EndComp
 Text GLabel 9250 4850 2    50   Input ~ 0
-CAM0_onboard_CLK
+CAM0_onboard_IO1
 $Comp
 L Device:L_Core_Iron L5
@@
 CAM1_DP0
 Text GLabel 14850 6850 0    50   Input ~ 0
-CAM1_CK
+CAM1_IO1
 Text GLabel 14850 6950 0    50   Input ~ 0
 CAM1_IO0
@@
 CM_3V3
 Text GLabel 17500 2000 0    50   Input ~ 0
-SDA
+CD0_SDA
 Text GLabel 17500 2150 0    50   Input ~ 0
-SCL
-Text GLabel 20900 1550 1    50   Input ~ 0
 CD0_SCL
-Text GLabel 17500 2900 0    50   Input ~ 0
-CAM0_CK
-Text GLabel 17500 3050 0    50   Input ~ 0
+Text GLabel 21450 1550 0    50   Input ~ 0
+CD0_SCL
+Text GLabel 17500 2600 0    50   Input ~ 0
+CAM0_IO1
+Text GLabel 17500 2750 0    50   Input ~ 0
 CAM0_IO0
 Text GLabel 17500 3350 0    50   Input ~ 0
@@
 Text GLabel 21450 4200 0    50   Input ~ 0
 SPI0_CS
-Text GLabel 20450 1650 0    50   Input ~ 0
-SDA
-Text GLabel 20450 1750 0    50   Input ~ 0
-SCL
 Text GLabel 21450 3400 0    50   Input ~ 0
 SDA
@@
 	16650 9350 16650 11600
 $Comp
-L Device:LED D4
-U 1 1 5E8BEF3F
-P 13500 13250
-F 0 "D4" V 13538 13133 50  0000 R CNN
-F 1 "LED" V 13447 13133 50  0000 R CNN
-F 2 "LEDs:LED_0805_HandSoldering" H 13500 13250 50  0001 C CNN
-F 3 "~" H 13500 13250 50  0001 C CNN
-	1    13500 13250
-	0    -1   -1   0
-$EndComp
-$Comp
-L Device:LED D5
-U 1 1 5E8BF370
-P 13700 13250
-F 0 "D5" V 13738 13133 50  0000 R CNN
-F 1 "LED" V 13647 13133 50  0000 R CNN
-F 2 "LEDs:LED_0805_HandSoldering" H 13700 13250 50  0001 C CNN
-F 3 "~" H 13700 13250 50  0001 C CNN
-	1    13700 13250
-	0    -1   -1   0
-$EndComp
-$Comp
 L Device:LED D7
 U 1 1 5E8BF46E
@@
 $EndComp
 Wire Wire Line
-	13500 13400 13500 13650
-Wire Wire Line
-	13500 13650 13700 13650
-Wire Wire Line
-	13700 13400 13700 13650
-Connection ~ 13700 13650
-Wire Wire Line
-	13700 13650 13900 13650
-Wire Wire Line
 	13900 13400 13900 13650
-Connection ~ 13900 13650
 Wire Wire Line
 	14100 13400 14100 13650
@@
 Text GLabel 15200 14500 1    50   Input ~ 0
 GPIO43
-Text GLabel 13500 12800 1    50   Input ~ 0
-GPIO28
-Text GLabel 13700 12800 1    50   Input ~ 0
-GPIO29
 Wire Notes Line
 	13200 11900 15850 11900
@@
 CAM1_DP0
 Text GLabel 11150 8350 2    50   Input ~ 0
-CAM1_CK
+CAM1_IO1
 Text GLabel 11150 8250 2    50   Input ~ 0
 CAM1_IO0
@@
 CAM0_DN1
 Text GLabel 5100 9400 0    50   Input ~ 0
-CAM0_CK
+CAM0_IO1
 Text GLabel 6500 8500 2    50   Input ~ 0
 CAM0_IO0
@@
 CAM0_onboard_DN1
 Text GLabel 6500 9400 2    50   Input ~ 0
-CAM0_onboard_CLK
+CAM0_onboard_IO1
 Text GLabel 5100 8400 0    50   Input ~ 0
 CAM0_onboard_IO0
@@
 CAM0_offboard_DN1
 Text GLabel 6500 9500 2    50   Input ~ 0
-CAM0_offboard_CK
+CAM0_offboard_IO1
 Text GLabel 5100 8500 0    50   Input ~ 0
 CAM0_offboard_IO0
@@
 CAM0_offboard_DN1
 Text GLabel 8250 8700 2    50   Input ~ 0
-CAM0_offboard_CK
+CAM0_offboard_IO1
 Text GLabel 8250 8600 2    50   Input ~ 0
 CAM0_offboard_IO0
@@
 CAM0_offboard_DN1
 Text GLabel 8900 9600 0    50   Input ~ 0
-CAM0_offboard_CK
+CAM0_offboard_IO1
 Text GLabel 8900 9700 0    50   Input ~ 0
 CAM0_offboard_IO0
@@
 $EndComp
 $Comp
-L Device:R R26
-U 1 1 5E57101C
-P 13700 12950
-F 0 "R26" H 13770 12996 50  0000 L CNN
-F 1 "470R" H 13770 12905 50  0000 L CNN
-F 2 "Resistors_SMD:R_0603_HandSoldering" V 13630 12950 50  0001 C CNN
-F 3 "~" H 13700 12950 50  0001 C CNN
-	1    13700 12950
-	1    0    0    -1
-$EndComp
-$Comp
-L Device:R R23
-U 1 1 5E571022
-P 13500 12950
-F 0 "R23" H 13570 12996 50  0000 L CNN
-F 1 "470R" H 13570 12905 50  0000 L CNN
-F 2 "Resistors_SMD:R_0603_HandSoldering" V 13430 12950 50  0001 C CNN
-F 3 "~" H 13500 12950 50  0001 C CNN
-	1    13500 12950
-	1    0    0    -1
-$EndComp
-$Comp
 L Device:R R41
 U 1 1 5E6A1A4F
@@
 	1    0    0    -1
 $EndComp
-$Comp
-L Connector_Generic:Conn_01x05 J11
-U 1 1 5C7AB2A0
-P 21650 3500
-F 0 "J11" H 21730 3542 50  0000 L CNN
-F 1 "Conn_01x05" H 21730 3451 50  0000 L CNN
-F 2 "Pin_Headers:Pin_Header_Straight_1x05_Pitch2.54mm" H 21650 3500 50  0001 C CNN
-F 3 "~" H 21650 3500 50  0001 C CNN
-	1    21650 3500
-	1    0    0    -1
-$EndComp
 Text GLabel 21450 3300 0    50   Input ~ 0
 3V3
@@
 L power:GND #PWR0172
 U 1 1 5C810D55
-P 21450 3700
-F 0 "#PWR0172" H 21450 3450 50  0001 C CNN
-F 1 "GND" H 21455 3527 50  0000 C CNN
-F 2 "" H 21450 3700 50  0001 C CNN
-F 3 "" H 21450 3700 50  0001 C CNN
-	1    21450 3700
+P 21450 3600
+F 0 "#PWR0172" H 21450 3350 50  0001 C CNN
+F 1 "GND" H 21455 3427 50  0000 C CNN
+F 2 "" H 21450 3600 50  0001 C CNN
+F 3 "" H 21450 3600 50  0001 C CNN
+	1    21450 3600
 	1    0    0    -1
 $EndComp
@@
 Wire Wire Line
 	19700 2600 19200 2600
-Text GLabel 19200 2750 2    50   Input ~ 0
-GPIO28
-Text GLabel 19200 2900 2    50   Input ~ 0
-GPIO29
 NoConn ~ 19200 5150
 NoConn ~ 19200 5300
@@
 	19850 11150 20350 11150
 Connection ~ 19850 11150
-Text GLabel 20350 11050 2    50   Input ~ 0
+Text GLabel 17500 10950 2    50   Input ~ 0
 ID_SD
-Text GLabel 20350 11150 2    50   Input ~ 0
+Text GLabel 17500 11100 2    50   Input ~ 0
 ID_SC
 $Comp
@@
 Wire Wire Line
 	20150 11550 20150 11450
-Wire Wire Line
-	20450 1650 20800 1650
-Wire Wire Line
-	20450 1750 20700 1750
-Wire Wire Line
-	21200 1550 21200 1650
-Wire Wire Line
-	21200 1650 21450 1650
-Connection ~ 21200 1650
-Wire Wire Line
-	21100 1550 21100 1750
-Wire Wire Line
-	21100 1750 21450 1750
-Connection ~ 21100 1750
 Text GLabel 17500 2300 0    50   Input ~ 0
-CAM1_CLK
+CAM1_IO1
 Text GLabel 17500 2450 0    50   Input ~ 0
 CAM1_IO0
-Text GLabel 21000 1550 1    50   Input ~ 0
+Text GLabel 21450 1450 0    50   Input ~ 0
 CD0_SDA
 Wire Wire Line
-	20900 1550 20900 1750
-Connection ~ 20900 1750
-Wire Wire Line
-	20900 1750 21100 1750
-Wire Wire Line
-	21000 1550 21000 1650
-Connection ~ 21000 1650
-Wire Wire Line
-	21000 1650 21200 1650
-Text GLabel 20800 1550 1    50   Input ~ 0
-ID_SD
-Text GLabel 20700 1550 1    50   Input ~ 0
-ID_SC
-Wire Wire Line
-	20800 1550 20800 1650
-Connection ~ 20800 1650
-Wire Wire Line
-	20800 1650 21000 1650
-Wire Wire Line
-	20700 1550 20700 1750
-Connection ~ 20700 1750
-Wire Wire Line
-	20700 1750 20900 1750
-$Comp
-L Connector_Generic:Conn_01x06 J?
-U 1 1 608AFE80
-P 21650 1850
-F 0 "J?" H 21730 1842 50  0000 L CNN
-F 1 "Conn_01x06" H 21730 1751 50  0000 L CNN
-F 2 "" H 21650 1850 50  0001 C CNN
-F 3 "~" H 21650 1850 50  0001 C CNN
-	1    21650 1850
-	1    0    0    -1
-$EndComp
-Wire Wire Line
 	19950 6300 20000 6300
 Connection ~ 20000 6300
@@
 Text Notes 19050 12550 0    197  ~ 0
 MOUNTING HOLES
+Text GLabel 19200 2750 2    50   Input ~ 0
+SDA
+Text GLabel 19200 2900 2    50   Input ~ 0
+SCL
+Text GLabel 17400 10950 0    50   Input ~ 0
+CD0_SDA
+Text GLabel 17400 11100 0    50   Input ~ 0
+CD0_SCL
+Wire Wire Line
+	17400 10950 17500 10950
+Wire Wire Line
+	17500 11100 17400 11100
+$Comp
+L Connector_Generic:Conn_01x08 J?
+U 1 1 5E0A8339
+P 21650 1750
+F 0 "J?" H 21730 1742 50  0000 L CNN
+F 1 "Conn_01x08" H 21730 1651 50  0000 L CNN
+F 2 "" H 21650 1750 50  0001 C CNN
+F 3 "~" H 21650 1750 50  0001 C CNN
+	1    21650 1750
+	1    0    0    -1
+$EndComp
+$Comp
+L Connector_Generic:Conn_01x04 J?
+U 1 1 5E227C53
+P 21650 3400
+F 0 "J?" H 21730 3392 50  0000 L CNN
+F 1 "Conn_01x04" H 21730 3301 50  0000 L CNN
+F 2 "Pin_Headers:Pin_Header_Straight_1x04_Pitch2.54mm" H 21650 3400 50  0001 C CNN
+F 3 "~" H 21650 3400 50  0001 C CNN
+	1    21650 3400
+	1    0    0    -1
+$EndComp
 $EndSCHEMATC

Commit message: A few small changes and fixes
Parts:
- removed D?: D_Zener, 5.6V, symbol Device:D_Zener
- removed J?: Conn_01x08, symbol Connector_Generic:Conn_01x08
- removed Q? (x2): Q_NPN_BCE, symbol Device:Q_NPN_BCE
- removed R1: 0R, Resistors_SMD:R_0603_HandSoldering, symbol Device:R
- removed R?: R, 1k, symbol Device:R
- added D? (x2): Q_SCR_AGK, symbol Device:Q_SCR_AGK
- added D?: D_Zener, 5.6V, symbol Device:D_Zener
- added F?: 2A Polyfuse, Inductors_SMD:L_1812_HandSoldering, symbol Device:Polyfuse
- added R?: R, 1k, symbol Device:R
Connections:
- net labels added: SCL1, SDA1
- net labels removed: SCL, SDA
- wire segments 582 -> 587
- no-connect marks 62 -> 65
Other:
- note added: "NEED TO PICK SUITABLE \nSCR THYRISTER AND \nUPDATE PINOUT ALSO \nCHECK FUSE SAME FOR \nUSB SECTION"
- moved on the sheet: D?, R?

Commit message: V1 routed ready for review
Parts:
- removed C6, C7: 100n, Capacitors_SMD:C_0603_HandSoldering, symbol Device:C
- removed J16: Conn_01x02, Socket_Strips:Socket_Strip_Straight_1x02_Pitch2.54mm, symbol Connector_Generic:Conn_01x02
- removed J3, J6: Conn_01x15, SFW15R-1STE1LF:AMPHENOL_SFW15R-1STE1LF, symbol Connector_Generic:Conn_01x15
- removed L1: L_Core_Iron, Inductors_SMD:L_0603_HandSoldering, symbol Device:L_Core_Iron
- removed R49: 0R, Resistors_SMD:R_0603_HandSoldering, symbol Device:R
- removed U3: LTC3406ES5-1.2, TO_SOT_Packages_SMD:TSOT-23-5_HandSoldering, symbol Regulator_Switching:LTC3406ES5-1.2
- removed U?: FST16233MTDX, symbol FST16233MTDX:FST16233MTDX
- added C34: 10u, Capacitor_SMD:C_0603_1608Metric_Pad1.05x0.95mm_HandSolder, symbol Device:C
- added D4: LED, LED_SMD:LED_0805_2012Metric_Pad1.15x1.40mm_HandSolder, symbol Device:LED
- added R23, R46: 10k, Resistor_SMD:R_0603_1608Metric_Pad1.05x0.95mm_HandSolder, symbol Device:R
- added R40, R42: 0R, Resistor_SMD:R_0603_1608Metric_Pad1.05x0.95mm_HandSolder, symbol Device:R
- added R48: 470R, Resistor_SMD:R_0603_1608Metric_Pad1.05x0.95mm_HandSolder, symbol Device:R
- added U14: AP3418, Package_TO_SOT_SMD:SOT-23-5_HandSoldering, symbol AP3418:AP3418
- added U15, U3: TS3DS10224, Package_DFN_QFN:QFN-20-1EP_3x3mm_P0.4mm_EP1.65x1.65mm_ThermalVias, symbol TS3DS10224:TS3DS10224
- added U16: 74LCX257MTC, Package_SO:TSSOP-16_4.4x5mm_P0.65mm, symbol TS3DS10224:74LCX257MTC
- C1, C12, C2, C22, C23, C28, C29, C33: value 47u -> 10u; footprint Capacitors_SMD:C_0603_HandSoldering -> Capacitor_SMD:C_0603_1608Metric_Pad1.05x0.95mm_HandSolder
- C10, C11, C13, C14, C15, C16, C17, C18, C19, C20, C21, C24, C25, C26, C27, C3, C30, C31, C4, C5, C8, C9: footprint Capacitors_SMD:C_0603_HandSoldering -> Capacitor_SMD:C_0603_1608Metric_Pad1.05x0.95mm_HandSolder
- C32: value 100nf -> 100n; footprint Capacitors_SMD:C_0603_HandSoldering -> Capacitor_SMD:C_0603_1608Metric_Pad1.05x0.95mm_HandSolder
- D1, D5: renamed from D?; value D_Zener -> 5.1V; footprint 5.6V -> Diode_SMD:D_SOD-123
- D10, D2: renamed from D?; footprint (none) -> Package_TO_SOT_SMD:TO-252-2; symbol Device:Q_SCR_AGK -> Device:Q_SCR_KAG
- D13, D6: footprint LEDs:LED_RGB_PLCC-6 -> LED_SMD:LED_RGB_PLCC-6
- D16, D3, D7, D8, D9: footprint LEDs:LED_0805_HandSoldering -> LED_SMD:LED_0805_2012Metric_Pad1.15x1.40mm_HandSolder
- F1: footprint Inductors_SMD:L_1812_HandSoldering -> Inductor_SMD:L_1812_4532Metric_Pad1.30x3.40mm_HandSolder
- F2: renamed from F?; footprint Inductors_SMD:L_1812_HandSoldering -> Inductor_SMD:L_1812_4532Metric_Pad1.30x3.40mm_HandSolder
- H1, H2, H3, H4: footprint Mounting_Holes:MountingHole_2.2mm_M2_DIN965_Pad -> MountingHole:MountingHole_3.2mm_M3
- J10: footprint Pin_Headers:Pin_Header_Straight_1x04_Pitch2.54mm -> Connector_PinHeader_2.54mm:PinHeader_1x04_P2.54mm_Vertical
- J12: footprint Pin_Headers:Pin_Header_Straight_1x06_Pitch2.54mm -> Connector_PinHeader_2.54mm:PinHeader_1x06_P2.54mm_Vertical
- J13, J7: footprint Pin_Headers:Pin_Header_Straight_1x02_Pitch2.54mm -> Connector_PinHeader_2.54mm:PinHeader_1x02_P2.54mm_Vertical
- J17, J2: footprint Connectors_USB:USB_Micro-B_Wuerth-629105150521 -> Connector_USB:USB_Micro-B_Amphenol_10103594-0001LF_Horizontal
- J18: footprint Pin_Headers:Pin_Header_Straight_1x03_Pitch2.54mm -> Connector_PinHeader_2.54mm:PinHeader_1x03_P2.54mm_Vertical
- J19, J20, J21, J22, J23: footprint Socket_Strips:Socket_Strip_Straight_1x02_Pitch2.54mm -> Connector_PinHeader_2.54mm:PinHeader_1x02_P2.54mm_Vertical
- J24: footprint Pin_Headers:Pin_Header_Straight_1x05_Pitch2.54mm -> Connector_PinHeader_2.54mm:PinHeader_1x05_P2.54mm_Vertical
- J3: renamed from J?; footprint (none) -> Connector_PinHeader_2.54mm:PinHeader_1x02_P2.54mm_Vertical
- J4: footprint DF37NC-30DS-0.4V_53_:HRS_DF37NC-30DS-0.4V(53) -> camera connector:HRS_DF37NC-30DS-0.4V(53)
- J5, J8, J9: footprint HDMI connector:WURTH_685119136923 -> mini_hdmi:CNC_2001-1-2-21-00-BK
- J6: renamed from J?; footprint Pin_Headers:Pin_Header_Straight_1x04_Pitch2.54mm -> Connector_PinHeader_2.54mm:PinHeader_1x04_P2.54mm_Vertical
- L12, L3, L5: footprint Inductors_SMD:L_0603_HandSoldering -> Inductor_SMD:L_0603_1608Metric_Pad1.05x0.95mm_HandSolder
- L2, L4: footprint Inductors_SMD:L_0805_HandSoldering -> Inductor_SMD:L_0805_2012Metric_Pad1.15x1.40mm_HandSolder
- Q10, Q12, Q8: footprint TO_SOT_Packages_SMD:SOT-23_Handsoldering -> Package_TO_SOT_SMD:SOT-23_Handsoldering
- Q2, Q3, Q4, Q5, Q6: renamed from Q?; footprint SOT323 -> DMG1012UW-7:SOT323
- R1, R26: renamed from R?; value R -> 1k; footprint 1k -> Resistor_SMD:R_0603_1608Metric_Pad1.05x0.95mm_HandSolder
- R10, R11, R12, R13, R16, R2, R21, R22, R24, R25, R27, R28, R29, R3, R30, R31, R32, R34, R36, R38, R39, R4, R41, R43, R44, R45, R5, R51, R52, R53, R54, R55, R56, R57, R58, R59, R7, R8, R9: footprint Resistors_SMD:R_0603_HandSoldering -> Resistor_SMD:R_0603_1608Metric_Pad1.05x0.95mm_HandSolder
- R14, R15, R17, R18, R6: value 0R -> NF; footprint Resistors_SMD:R_0603_HandSoldering -> Resistor_SMD:R_0603_1608Metric_Pad1.05x0.95mm_HandSolder
- R19, R20: value 1.75K -> 1.8K; footprint Resistors_SMD:R_0603_HandSoldering -> Resistor_SMD:R_0603_1608Metric_Pad1.05x0.95mm_HandSolder
- R33, R35, R37: renamed from R?; footprint (none) -> Resistor_SMD:R_0603_1608Metric_Pad1.05x0.95mm_HandSolder
- SW1: footprint Buttons_Switches_THT:SW_Tactile_Straight_KSL0Axx1LFTR -> Button_Switch_THT:SW_Tactile_Straight_KSL0Axx1LFTR
- U1: footprint TO_SOT_Packages_SMD:SOT-23-6_Handsoldering -> Package_TO_SOT_SMD:SOT-23-6_Handsoldering
- U10: footprint TO_SOT_Packages_SMD:SOT-23-6 -> Package_TO_SOT_SMD:SOT-23-6_Handsoldering
- U5, U9: footprint TO_SOT_Packages_SMD:SOT-23-5_HandSoldering -> Package_TO_SOT_SMD:SOT-23-5_HandSoldering
- U6: footprint TO_SOT_Packages_SMD:SOT-666 -> Package_TO_SOT_SMD:SOT-666
- U7: footprint Housings_LGA:Bosch_LGA-14_3x2.5mm_Pitch0.5mm -> Package_LGA:Bosch_LGA-14_3x2.5mm_P0.5mm
- U8: footprint Crystals:Crystal_SMD_2016-4pin_2.0x1.6mm -> Crystal:Crystal_SMD_2016-4Pin_2.0x1.6mm
- gave numbers to parts that had none: 1
- renumbered Q11 to Q9
Connections:
- net CAM0_onboard_CLK is gone; now on net CAM0_onboard_DP0: J4.24 (Pin_24)
- net TVDAC is gone; now on net CM_3V3: MD1.166 (TVDAC)
- net 1V2: now also C28.1, J4.4 (Pin_4), C34.1, R23.1; no longer J4.27 (Pin_27)
- net 2V8: now also J4.10 (Pin_10); no longer J4.21 (Pin_21)
- net 3V3: now also U15.10 (ENB), U15.12 (SBI), U15.13 (VCC), U15.14 (SAI), U15.16 (ENA), U16.16 (VCC), U3.10 (ENB), U3.12 (SBI), U3.13 (VCC), U3.14 (SAI), U3.16 (ENA)
- net 5V: now also Q9.5 (E), R48.1, U14.4 (VIN); no longer Q9.6 (E)
- net CAM0_CN: now also U15.2 (INA-)
- net CAM0_CP: now also U15.1 (INA+)
- net CAM0_DN0: now also U3.2 (INA-)
- net CAM0_DN1: now also U15.4 (INB-)
- net CAM0_DP0: now also U3.1 (INA+)
- net CAM0_DP1: now also U15.3 (INB+)
- net CAM0_IO0: now also U16.9 (Zd)
- net CAM0_IO1: now also U16.12 (Zc)
- net CAM0_offboard_CN: now also U15.19 (OUTA1-)
- net CAM0_offboard_CP: now also U15.20 (OUTA1+)
- net CAM0_offboard_DN0: now also U3.19 (OUTA1-)
- net CAM0_offboard_DN1: now also U15.7 (OUTB1-)
- net CAM0_offboard_DP0: now also U3.20 (OUTA1+)
- net CAM0_offboard_DP1: now also U15.6 (OUTB1+)
- net CAM0_offboard_IO0: now also U16.10 (I1d)
- net CAM0_offboard_IO1: now also U16.14 (I0C)
- net CAM0_onboard_CN: now also J4.26 (Pin_26), U15.17 (OUTA0-); no longer J4.5 (Pin_5)
- net CAM0_onboard_CP: now also J4.27 (Pin_27), U15.18 (OUTA0+); no longer J4.4 (Pin_4)
- net CAM0_onboard_DN0: now also J4.23 (Pin_23), U3.17 (OUTA0-); no longer J4.8 (Pin_8)
- net CAM0_onboard_DN1: now also J4.20 (Pin_20), U15.9 (OUTB0-); no longer J4.11 (Pin_11)
- net CAM0_onboard_DP0: now also U3.18 (OUTA0+); no longer J4.7 (Pin_7)
- net CAM0_onboard_DP1: now also J4.21 (Pin_21), U15.8 (OUTB0+); no longer J4.10 (Pin_10)
- net CAM0_onboard_IO0: now also U14.1 (EN), U16.11 (eI0d)
- net CAM0_onboard_IO1: now also J4.7 (Pin_7), U16.13 (I1C)
- net CAM0_onboard_n: now also U15.11 (SBO), U15.15 (SAO), U16.1 (S), U3.15 (SAO)
- net CAM_1V8: now also J4.3 (Pin_3), J4.5 (Pin_5); no longer J4.26 (Pin_26), J4.28 (Pin_28)
- net CD0_SCL: now also U16.7 (Zb)
- net CD0_SDA: now also U16.4 (Za)
- net CD0_offboard_SCL: now also U16.6 (I1b)
- net CD0_offboard_SDA: now also U16.3 (I1a)
- net CD0_onboard_SCL: now also U16.5 (I0b)
- net CD0_onboard_SDA: now also U16.2 (I0a)
- net GND: now also D10.1 (K), D2.1 (K), J4.28 (Pin_28), J4.8 (Pin_8), C34.2, D4.1 (K), R40.2, R42.2, R46.2, U14.2 (GND), U15.21 (Thermal_pad), U15.5 (GND), U16.15 (OE), U16.8 (GND), U3.21 (Thermal_pad), U3.5 (GND); no longer D10.3 (K), D2.3 (K), J4.23 (Pin_23), J4.3 (Pin_3), U7.2 (SDX), U7.3 (SCX)
- net ID_SC: now also R35.2, U13.6 (SCL)
- net ID_SD: now also R33.2, U13.5 (SDA)
- net at R7.1, U6.1: now also J4.29 (Pin_29); no longer J4.2 (Pin_2)
- net at R11.2, U6.4: now also J4.30 (Pin_30); no longer J4.1 (Pin_1)
- net at L3.1: now also U14.3 (SW)
- net at D1.1 (K), F1.1, Q1.6 (E)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: now also D2.2 (A); no longer D2.1 (A)
- net at Q12.1 (G), R59.1: now also Q9.4 (C); no longer Q9.1 (C)
- net at D5.1 (K), J13.2 (Pin_2), Q12.3 (D)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: now also D10.2 (A); no longer D10.1 (A)
- net at Q9.1 (C), Q9.2 (B), R58.1: now also Q9.3 (B); no longer Q9.2 (B)
- net at D1.2 (A), R1.1: now also D2.3 (G); no longer D2.2 (G)
- net at J13.1 (Pin_1): now also F2.2
- net at D5.2 (A), R26.1: now also D10.3 (G); no longer D10.2 (G)
- net GPIO12: no longer names the net of MD1.45 (GPIO12)
- net GPIO13: no longer names the net of MD1.47 (GPIO13)
- net GPIO21: no longer names the net of MD1.71 (GPIO21)
- net GPIO22: no longer names the net of MD1.75 (GPIO22)
- net GPIO23: no longer names the net of MD1.77 (GPIO23)
- net GPIO24: no longer names the net of MD1.81 (GPIO24)
- net GPIO25: no longer names the net of MD1.83 (GPIO25)
- net GPIO26: no longer names the net of MD1.87 (GPIO26)
- net GPIO33: no longer names the net of MD1.48 (GPIO33)
- net GPIO34: no longer names the net of MD1.52 (GPIO34)
- net GPIO35: no longer names the net of MD1.54 (GPIO35)
- net GPIO36: no longer names the net of MD1.58 (GPIO36)
- net GPIO37: no longer names the net of MD1.60 (GPIO37)
- net USB_DM renamed USB_D-
- net USB_DP renamed USB_D+
- net VBUSA renamed VBUS_A
- net VBUS_A: no longer C28.1
- net VBUSB renamed VBUS_B
- new net: R40.1, U7.2 (SDX)
- new net: R42.1, U7.3 (SCX)
- new net: D4.2 (A), R48.2
- new net: R23.2, R46.1, U14.5 (FB)
- no-connect marks 65 -> 75
Other:
- note added: "NEED TO CHECK \nHDMI FOOTPRINT"
- note removed: "NEED TO PICK SUITABLE \nSCR THYRISTER AND \nUPDATE PINOUT ALSO \nCHECK FUSE SAME FOR \nUSB SECTION"
- moved on the sheet: C11, C16, C25, L12, L3, R12, R3, R44, U9
